File: PCB/AntennaSwitch_6x2/Interlock.sch (KiCad schematic (older format))
At the start: 80 parts, among them J1 Conn_01x08, J2 Conn_01x08, J3 Conn_01x08, Q1 2N7002K, SW1 LOAD, SW2 SRBV170501, SW3 SRBV170501, SW4 M/R, U1 74HC238, U10 74HC148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

Commit message: manufacturing files
Parts:
- R38, R39, R40, R41, R42, R43, R44, R45, R46, R47, R48, R49, R50, R51: value 81 -> 33
- U1, U10, U11, U12, U13, U4: footprint Housings_SOIC:SOIC-16_3.9x9.9mm_Pitch1.27mm -> digikey-footprints:SOIC-16_W3.90mm
- U14, U15: value Blue 0.59'' -> Blue 0.56'' CC
- U2, U3: footprint Housings_SOIC:SOIC-20W_7.5x12.8mm_Pitch1.27mm -> MyPCBLib:SOIC-20_W7.5mm
- U5, U6, U7, U8: footprint Housings_SOIC:SOIC-14_3.9x8.7mm_Pitch1.27mm -> digikey-footprints:SOIC-14_W3.9mm

Commit message: FS Tools
Parts:
- Q1: value 2N7002K -> 2N7002; footprint TO_SOT_Packages_SMD:SOT-23 -> lc_lib:SOT-23(SOT-23-3)
Connections:
- net REMOTE2_0 is gone; now on net REMOTE2_1: R33.2, U4.14 (O1)
- net REMOTE1_1: now also R32.1; no longer R30.1, U1.13 (O2)
- net REMOTE1_2: now also R30.1, U1.13 (O2); no longer R28.1, U1.12 (O3)
- net REMOTE1_3: now also R28.1, U1.12 (O3); no longer R26.1, U1.11 (O4)
- net REMOTE1_4: now also R26.1, U1.11 (O4); no longer R24.1, U1.10 (O5)
- net REMOTE1_5: now also R24.1, U1.10 (O5); no longer R22.1, U1.9 (O6)
- net REMOTE2_1: no longer R31.2, U4.13 (O2)
- net REMOTE2_2: now also R31.2, U4.13 (O2); no longer R29.2, U4.12 (O3)
- net REMOTE2_3: now also R29.2, U4.12 (O3); no longer R27.2, U4.11 (O4)
- net REMOTE2_4: now also R27.2, U4.11 (O4); no longer R25.2, U4.10 (O5)
- net REMOTE2_5: now also R25.2, U4.10 (O5); no longer R23.2, U4.9 (O6)
- net REMOTE1_0 renamed REMOTE1_
- net REMOTE1_: no longer R32.1
- new net REMOTE1_6: R22.1, U1.9 (O6)
- new net REMOTE2_6: R23.2, U4.9 (O6)
Changed lines of the file:
@@
 $EndComp
 Text Label 1600 5500 1    50   ~ 0
-REMOTE1_0
+REMOTE1_
 Text Label 1700 5500 1    50   ~ 0
-REMOTE1_1
+REMOTE1_2
 Text Label 1800 5500 1    50   ~ 0
-REMOTE1_2
+REMOTE1_3
 Text Label 1900 5500 1    50   ~ 0
-REMOTE1_3
+REMOTE1_4
 Text Label 2000 5500 1    50   ~ 0
-REMOTE1_4
+REMOTE1_5
 Text Label 2100 5500 1    50   ~ 0
-REMOTE1_5
+REMOTE1_6
 Text Label 3450 5500 1    50   ~ 0
-REMOTE2_0
+REMOTE2_1
 Text Label 3550 5500 1    50   ~ 0
-REMOTE2_1
+REMOTE2_2
 Text Label 3650 5500 1    50   ~ 0
-REMOTE2_2
+REMOTE2_3
 Text Label 3750 5500 1    50   ~ 0
-REMOTE2_3
+REMOTE2_4
 Text Label 3850 5500 1    50   ~ 0
-REMOTE2_4
+REMOTE2_5
 Text Label 3950 5500 1    50   ~ 0
-REMOTE2_5
+REMOTE2_6
 Text Notes 1300 5850 1    50   ~ 0
 HIGH effective\n
@@
 	3450 4050 3450 3950
 Text Label 4150 2350 3    50   ~ 0
-REMOTE1_0
+REMOTE1_1
 Text Label 4050 2350 3    50   ~ 0
-REMOTE1_1
+REMOTE1_2
 Text Label 3950 2350 3    50   ~ 0
-REMOTE1_2
+REMOTE1_3
 Text Label 3850 2350 3    50   ~ 0
-REMOTE1_3
+REMOTE1_4
 Text Label 3750 2350 3    50   ~ 0
-REMOTE1_4
+REMOTE1_5
 Text Label 3650 2350 3    50   ~ 0
-REMOTE1_5
+REMOTE1_6
 $Comp
 L power:GND #PWR018
@@
 $EndComp
 Text Label 4150 4450 3    50   ~ 0
-REMOTE2_0
+REMOTE2_1
 Text Label 4050 4450 3    50   ~ 0
-REMOTE2_1
+REMOTE2_2
 Text Label 3950 4450 3    50   ~ 0
-REMOTE2_2
+REMOTE2_3
 Text Label 3850 4450 3    50   ~ 0
-REMOTE2_3
+REMOTE2_4
 Text Label 3750 4450 3    50   ~ 0
-REMOTE2_4
+REMOTE2_5
 Text Label 3650 4450 3    50   ~ 0
-REMOTE2_5
+REMOTE2_6
 Wire Wire Line
 	3450 3850 3550 3850
@@
 P 6650 5150
 F 0 "Q1" H 6450 5400 50  0000 L CNN
-F 1 "2N7002K" H 6350 5300 50  0000 L CNN
-F 2 "TO_SOT_Packages_SMD:SOT-23" H 6850 5075 50  0001 L CIN
+F 1 "2N7002" H 6350 5300 50  0000 L CNN
+F 2 "lc_lib:SOT-23(SOT-23-3)" H 6850 5075 50  0001 L CIN
 F 3 "https://www.fairchildsemi.com/datasheets/2N/2N7002.pdf" H 6650 5150 50  0001 L CNN
 	1    6650 5150
