File: PCB/AntennaSwitch_6x2/Remote.sch (KiCad schematic (older format))
At the start: 61 parts, among them J4 HR913550A, J5 SWD, J6 485, J8 Conn_01x01, SW5 RESET, U16 STM32F030F4Px, U17 MAX485E, U18 CH395Q, U19 AZ1117-1.8, Y1 30MHz

Commit message: manufacturing files
Parts:
- U17: footprint Housings_SOIC:SOIC-8_3.9x4.9mm_Pitch1.27mm -> digikey-footprints:SOIC-8_W3.9mm
Other:
- note added: "BCD Monitoring Port"
Changed lines of the file:
@@
 F 0 "U17" H 4000 7250 50  0000 C CNN
 F 1 "MAX485E" H 4000 7150 50  0000 C CNN
-F 2 "Housings_SOIC:SOIC-8_3.9x4.9mm_Pitch1.27mm" H 4200 5950 50  0001 C CNN
+F 2 "digikey-footprints:SOIC-8_W3.9mm" H 4200 5950 50  0001 C CNN
 F 3 "https://datasheets.maximintegrated.com/en/ds/MAX1487E-MAX491E.pdf" H 4200 6700 50  0001 C CNN
 	1    4200 6650
@@
 Wire Wire Line
 	2850 2300 2850 2550
+Text Notes 8500 4100 0    50   ~ 0
+BCD Monitoring Port
 $EndSCHEMATC

Commit message: FS Tools
Parts:
- C8, C9: value 20pF -> 10pF
- U16: footprint digikey-footprints:TSSOP-20_W4.4mm -> lc_lib:TSSOP-20
Changed lines of the file:
@@
 F 0 "U16" H 3400 2200 50  0000 C CNN
 F 1 "STM32F030F4Px" H 3400 2300 50  0000 C CNN
-F 2 "digikey-footprints:TSSOP-20_W4.4mm" H 3400 2350 50  0001 R CNN
+F 2 "lc_lib:TSSOP-20" H 3400 2350 50  0001 R CNN
 F 3 "http://www.st.com/st-web-ui/static/active/en/resource/technical/document/datasheet/DM00088500.pdf" H 3800 3050 50  0001 C CNN
 	1    3800 3050
@@
 P 5100 3700
 F 0 "C8" V 4871 3700 50  0000 C CNN
-F 1 "20pF" V 4962 3700 50  0000 C CNN
+F 1 "10pF" V 4962 3700 50  0000 C CNN
 F 2 "Capacitors_SMD:C_0603" H 5100 3700 50  0001 C CNN
 F 3 "~" H 5100 3700 50  0001 C CNN
@@
 P 5100 4000
 F 0 "C9" V 5200 4000 50  0000 C CNN
-F 1 "20pF" V 5300 4000 50  0000 C CNN
+F 1 "10pF" V 5300 4000 50  0000 C CNN
 F 2 "Capacitors_SMD:C_0603" H 5100 4000 50  0001 C CNN
 F 3 "~" H 5100 4000 50  0001 C CNN
