File: PCB/ControlBoard-2/AntennaSwitch_6x2 - Copy.kicad_pcb (KiCad board)
At the start: 2 copper layers, 84 x 90 mm, 147 parts, among them J1 Blaster JTAG, J3 Conn_01x08, J4 Conn_01x08, J5 HR913550A, J6 SWD, J7 485, J8 12VDC, Q1 8550, Q10 8050, Q11 8050, Q12 8050, Q13 8050, Q14 8050, Q15 8550, Q16 8550, Q17 8550, Q18 8550, Q19 8550, Q2 8550, Q20 8550, Q21 8550, Q22 8550, Q23 8550, Q24 8550, Q25 8550, Q26 8550, Q3 8050, Q4 8050, Q5 8050, Q6 8050, Q7 8050, Q8 8050, Q9 8050, SW1 SRBV170501, SW2 SRBV170501, SW3 LOAD, SW4 REMOTE, U1 EPM240T100, U3 AZ1117-1.8, U4 CH395Q, U5 STM32F030C8Tx, U6 MAX485E, U7 SY8303, U8 AZ1117-3.3, Y1 30MHz

Commit message: Control Board 2 routed
Parts:
- moved R1 17.6 mm to (72.5, 75.4), turned to 180 degrees
- moved R2 17.3 mm to (72.5, 77.8), turned to 180 degrees
- moved R8 17.2 mm to (72.5, 80.2), turned to 180 degrees
- moved R3 17.1 mm to (72.5, 82.6), turned to 180 degrees
- moved R5 17.0 mm to (72.5, 85.0), turned to 180 degrees
- moved R6 16.9 mm to (72.5, 73.0), turned to 180 degrees
- moved R7 12.9 mm to (72.5, 70.6)
- moved R12 9.52 mm to (88.5, 131.3), turned to 90 degrees
- moved R17 1.52 mm to (90.2, 131.3)
- moved C5 1.30 mm to (89.2, 111.5)
Connections:
- net Net-(R6-Pad2) renamed /Interlock/SEG1_F
- net Net-(R7-Pad2) renamed /Interlock/SEG1_G
- net Net-(SW1-Pad4) renamed /Interlock/SW1_2
- net Net-(SW1-Pad6) renamed /Interlock/SW1_4
- net Net-(SW1-Pad7) renamed /Interlock/SW1_5
- net Net-(SW1-Pad8) renamed /Interlock/SW1_6
- net Net-(SW2-Pad3) renamed /Interlock/SW2_1
- net Net-(SW2-Pad4) renamed /Interlock/SW2_2
- net Net-(SW2-Pad5) renamed /Interlock/SW2_3
- net Net-(SW2-Pad6) renamed /Interlock/SW2_4
- net Net-(SW2-Pad7) renamed /Interlock/SW2_5
- net Net-(SW2-Pad8) renamed /Interlock/SW2_6
- R1 pad 2: Net-(R1-Pad2) -> /Interlock/SEG1_A
- R10 pad 2: Net-(R10-Pad2) -> /Interlock/SEG1
- R11 pad 2: Net-(R11-Pad2) -> /Interlock/SEG2_B
- R12 pad 2: Net-(R12-Pad2) -> /Interlock/SEG2_C
- R13 pad 2: Net-(R13-Pad2) -> /Interlock/SEG2_D
- R14 pad 2: Net-(R14-Pad2) -> /Interlock/SEG2_E
- R15 pad 2: Net-(R15-Pad2) -> /Interlock/SEG2_F
- R16 pad 2: Net-(R16-Pad2) -> /Interlock/SEG2_G
- R17 pad 2: Net-(R17-Pad2) -> /Interlock/SEG2_DP
- R2 pad 2: Net-(R2-Pad2) -> /Interlock/SEG1_B
- R3 pad 2: Net-(R3-Pad2) -> /Interlock/SEG1_C
- R4 pad 2: Net-(R4-Pad2) -> /Interlock/SEG1_D
- R5 pad 2: Net-(R5-Pad2) -> /Interlock/SEG1_E
- R8 pad 2: Net-(R8-Pad2) -> /Interlock/SEG1_DP
- R9 pad 2: Net-(R9-Pad2) -> /Interlock/SEG2_A
- SEG1 pad 8: Net-(SEG1-Pad8) -> Net-(Q1-Pad3)
- SEG2 pad 8: Net-(SEG2-Pad8) -> Net-(Q2-Pad3)
- SW1 pad 3: Net-(SW1-Pad3) -> /Interlock/SW1_1
- SW1 pad 5: Net-(SW1-Pad5) -> /Interlock/SW1_3
- U1 pad 2: Net-(SW1-Pad3) -> /Interlock/SW1_3
- U1 pad 35: /Interlock/SEL1_1 -> /Interlock/SEL2_6
- U1 pad 36: /Interlock/SEL2_1 -> /Interlock/SEL1_6
- U1 pad 37: /Interlock/SEL1_2 -> /Interlock/SEL2_5
- U1 pad 38: /Interlock/SEL2_2 -> /Interlock/SEL1_5
- U1 pad 39: /Interlock/SEL1_3 -> /Interlock/SEL2_4
- U1 pad 4: Net-(SW1-Pad5) -> /Interlock/SW1_1
- U1 pad 40: /Interlock/SEL2_3 -> /Interlock/SEL1_4
- U1 pad 41: /Interlock/SEL1_4 -> /Interlock/SEL2_3
- U1 pad 42: /Interlock/SEL2_4 -> /Interlock/SEL1_3
- U1 pad 43: /Interlock/SEL1_5 -> /Interlock/SEL2_2
- U1 pad 44: /Interlock/SEL2_5 -> /Interlock/SEL1_2
- U1 pad 47: /Interlock/SEL1_6 -> /Interlock/SEL2_1
- U1 pad 48: /Interlock/SEL2_6 -> /Interlock/SEL1_1
- U1 pad 50: Net-(U1-Pad50) -> /Interlock/SEG1
- U1 pad 51: Net-(U1-Pad51) -> /Interlock/SEG1_D
- U1 pad 52: Net-(R1-Pad2) -> /Interlock/SEG1_E
- U1 pad 53: Net-(R2-Pad2) -> /Interlock/SEG1_C
- U1 pad 54: Net-(R3-Pad2) -> /Interlock/SEG1_DP
- U1 pad 55: Net-(R4-Pad2) -> /Interlock/SEG1_B
- U1 pad 56: Net-(R5-Pad2) -> /Interlock/SEG1_A
- U1 pad 61: Net-(R8-Pad2) -> Net-(U1-Pad61)
- U1 pad 66: Net-(R9-Pad2) -> /Interlock/SEG2_E
- U1 pad 67: Net-(R11-Pad2) -> /Interlock/SEG2_G
- U1 pad 68: Net-(R12-Pad2) -> /Interlock/SEG2_D
- U1 pad 69: Net-(R13-Pad2) -> /Interlock/SEG2_F
- U1 pad 70: Net-(R14-Pad2) -> /Interlock/SEG2_C
- U1 pad 71: Net-(R15-Pad2) -> /Interlock/SEG2_A
- U1 pad 72: Net-(R16-Pad2) -> /Interlock/SEG2_DP
- U1 pad 73: Net-(R17-Pad2) -> /Interlock/SEG2_B
- U1 pad 75: Net-(R10-Pad2) -> Net-(U1-Pad75)
Routing:
- net +12V: track 103.9 -> 281.3 mm
- net +3V3: track 420.4 -> 493.8 mm, vias 26 -> 42
- net /Interlock/SW1_3: track 0.00 -> 68.2 mm, vias 0 -> 4
- net /Interlock/SW1_2: track 0.00 -> 67.9 mm, vias 0 -> 4
- net /Interlock/SW1_1: track 0.00 -> 66.9 mm, vias 0 -> 4
- net /Interlock/SEL2_6: track 0.00 -> 61.7 mm, vias 0 -> 2
- net /Interlock/SEG1_G: track 0.00 -> 59.9 mm
- net /Interlock/SEL1_6: track 0.00 -> 57.8 mm, vias 0 -> 2
- net /Interlock/SEG1_F: track 0.00 -> 55.6 mm
- net /Interlock/SEL2_5: track 0.00 -> 54.7 mm, vias 0 -> 2
- net /Interlock/SEG1_A: track 0.00 -> 51.7 mm
- net /Interlock/SEL1_5: track 0.00 -> 50.7 mm, vias 0 -> 2
- net /Interlock/SEL2_4: track 0.00 -> 47.9 mm, vias 0 -> 2
- net /Interlock/SEG1_B: track 0.00 -> 47.7 mm
- net Net-(R18-Pad2): track 0.00 -> 45.5 mm, vias 0 -> 2
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- added copper zone on B.Cu, net +1V8
- added copper zone on F.Cu, net +1V8
- added copper zone on B.Cu, net +3V3
- added copper zone on F.Cu, net +3V3

Commit message: final
Parts:
- added C43: 104, lc_lib:0603_C, F.Cu at (70.3, 94.7)
- added J2: Conn_01x01, Connectors:PINTST, F.Cu at (123.5, 109.8)
- added J9: RST, Connectors:PINTST, F.Cu at (63.7, 96.5)
- added R19: 1K, lc_lib:0603_R, F.Cu at (66.6, 94.6)
- added R20: 0, lc_lib:1206_R, F.Cu at (93.0, 64.3)
- added R21: 47K, lc_lib:0603_R, F.Cu at (77.8, 144.8)
- added R22: 47K, lc_lib:0603_R, F.Cu at (82.1, 144.8)
- added R23: 47K, lc_lib:0603_R, F.Cu at (77.8, 147.6)
- added R24: 47K, lc_lib:0603_R, F.Cu at (98.5, 136.6)
- added R38: 47K, lc_lib:0603_R, F.Cu at (82.1, 147.6)
- added R39: 47K, lc_lib:0603_R, F.Cu at (86.4, 144.8)
- added R40: 47K, lc_lib:0603_R, F.Cu at (98.5, 139.4)
- added R41: 47K, lc_lib:0603_R, F.Cu at (90.6, 144.8)
- added R42: 47K, lc_lib:0603_R, F.Cu at (86.4, 147.6)
- added R43: 47K, lc_lib:0603_R, F.Cu at (90.6, 147.6)
- added R60: 47K, lc_lib:0603_R, F.Cu at (98.5, 142.2)
- added R61: 47K, lc_lib:0603_R, F.Cu at (94.9, 145.0)
- added U2: 74HC04, lc_lib:TSSOP-14, F.Cu at (81.1, 139.3)
- added U9: 74HC04, lc_lib:TSSOP-14, F.Cu at (91.5, 139.3)
- moved C10 5.71 mm to (111.5, 74.7)
- moved SC3 1.82 mm to (129.5, 110.6)
- moved R53 0.46 mm to (129.4, 97.8)
- moved F1 0.28 mm to (71.1, 62.7)
- moved D3 0.25 mm to (74.8, 63.8)
- moved U6 0.25 mm to (127.4, 103.1)
- moved C18 0.13 mm to (125.3, 78.1)
- moved R17 0.13 mm to (90.3, 131.3)
- moved C21 0.13 mm to (132.1, 101.5)
Connections:
- Q10 pad 1: /Interlock/SEL2_4 -> Net-(Q10-Pad1)
- Q11 pad 1: /Interlock/SEL1_5 -> Net-(Q11-Pad1)
- Q12 pad 1: /Interlock/SEL2_5 -> Net-(Q12-Pad1)
- Q13 pad 1: /Interlock/SEL1_6 -> Net-(Q13-Pad1)
- Q14 pad 1: /Interlock/SEL2_6 -> Net-(Q14-Pad1)
- Q3 pad 1: /Interlock/SEL1_1 -> Net-(Q3-Pad1)
- Q4 pad 1: /Interlock/SEL2_1 -> Net-(Q4-Pad1)
- Q5 pad 1: /Interlock/SEL1_2 -> Net-(Q5-Pad1)
- Q6 pad 1: /Interlock/SEL2_2 -> Net-(Q6-Pad1)
- Q7 pad 1: /Interlock/SEL1_3 -> Net-(Q7-Pad1)
- Q8 pad 1: /Interlock/SEL2_3 -> Net-(Q8-Pad1)
- Q9 pad 1: /Interlock/SEL1_4 -> Net-(Q9-Pad1)
- U1 pad 27: Net-(U1-Pad27) -> /Interlock/CPLDRST
- U8 pad 3: Net-(C38-Pad1) -> Net-(R20-Pad1)
Routing:
- net /Interlock/SW2_3: track 0.00 -> 81.5 mm, vias 0 -> 2
- net /Interlock/SW2_4: track 0.00 -> 56.1 mm, vias 0 -> 4
- net /Interlock/SW2_5: track 0.00 -> 54.1 mm, vias 0 -> 4
- net /Interlock/SW2_2: track 0.00 -> 52.6 mm, vias 0 -> 2
- net /Interlock/SW2_6: track 0.00 -> 50.4 mm, vias 0 -> 4
- net +3V3: track 493.8 -> 541.6 mm, vias 42 -> 47
- net /Interlock/LOAD: track 0.00 -> 43.1 mm, vias 0 -> 4
- net /Interlock/SW2_1: track 0.00 -> 41.1 mm, vias 0 -> 3
- net /Interlock/REMOTE: track 0.00 -> 22.7 mm, vias 0 -> 1
- net /Remote/RST: track 6.56 -> 29.0 mm, vias 0 -> 3
- net /Interlock/CPLDRST: track 0.00 -> 21.8 mm, vias 0 -> 2
- net Net-(Q1-Pad3): track 4.56 -> 21.5 mm
- net Net-(D1-Pad1): track 0.00 -> 15.5 mm
- net Net-(Q2-Pad3): track 10.1 -> 25.4 mm, vias 0 -> 1
- net BCD2_0: track 0.00 -> 9.71 mm
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- added copper zone on F.Cu, net Net-(R20-Pad1)
- added copper zone on F.Cu, net chasis
Other:
- net class +12V: clearance 0.254 -> 0.1524
- net class +3V3: clearance 0.254 -> 0.1524
- net class CH395_GPIO: clearance 0.2032 -> 0.1524
- net class CHASIS: clearance 0.508 -> 0.1524
- net class Default: clearance 0.2032 -> 0.1524
- net class RS485 added: clearance 0.508, trace_width 0.2032, via_dia 0.8, via_drill 0.4
- rule trace_clearance: 0.2032 -> 0.1524
- board text added: "+"
- board text added: "+Freq"
- board text added: "-"
- board text added: "12VDC"
- board text added: "3.3V"
- board text added: "485"
- board text added: "500kHz-2MHz"
- board text added: "6x2 Antenna Switch Control Board V0.2 w/ CPLD Interlock"
- board text added: "A"
- board text added: "B"
- board text added: "CLK"
- board text added: "CPLD RST"
- board text added: "Designed by: Lu, Zening BI4WOP 2019.11.01"
- board text added: "Ethernet"
- board text added: "Feel free to distribute, copy and modify this deisgn"
- board text added: "GND"
- board text added: "IO"
- board text added: "Load"
- board text added: "Power"
- board text added: "RST"
- board text added: "Remote"
- board text added: "SWD"
- board text added: "Zening's Radio Shack BI4WOP"
