File: PCB/ControlBoard-2/AntennaSwitch_6x2.kicad_pcb (KiCad board)
At the start: 2 copper layers, 84 x 90 mm, 148 parts, among them J1 Blaster JTAG, J3 Conn_01x08, J4 Conn_01x08, J5 HR913550A, J6 SWD, J7 485, J8 12VDC, Q1 8550, Q10 8050, Q11 8050, Q12 8050, Q13 8050, Q14 8050, Q15 8550, Q16 8550, Q17 8550, Q18 8550, Q19 8550, Q2 8550, Q20 8550, Q21 8550, Q22 8550, Q23 8550, Q24 8550, Q25 8550, Q26 8550, Q3 8050, Q4 8050, Q5 8050, Q6 8050, Q7 8050, Q8 8050, Q9 8050, SW1 SRBV170501, SW2 SRBV170501, SW3 LOAD, SW4 REMOTE, U1 EPM240T100, U3 AZ1117-1.8, U4 CH395Q, U5 STM32F030C8Tx, U6 MAX485E, U7 SY8303, U8 AZ1117-3.3, Y1 30MHz

Commit message: Control Board 2 routed
Parts:
- removed C27: 104, lc_lib:0603_C
- moved R12 9.52 mm to (88.5, 131.3), turned to 90 degrees
- moved R17 1.52 mm to (90.2, 131.3)
- moved C5 0.37 mm to (89.2, 111.5)
Connections:
- U1 pad 2: /Interlock/SW1_1 -> /Interlock/SW1_3
- U1 pad 4: /Interlock/SW1_3 -> /Interlock/SW1_1
Routing:
- net +12V: track 103.9 -> 281.5 mm
- net +3V3: track 420.1 -> 538.4 mm, vias 23 -> 46
- net /Interlock/SW2_3: track 0.00 -> 81.5 mm, vias 0 -> 2
- net /Interlock/SW1_3: track 0.00 -> 68.2 mm, vias 0 -> 4
- net /Interlock/SW1_2: track 0.00 -> 67.9 mm, vias 0 -> 4
- net /Interlock/SW1_1: track 0.00 -> 66.9 mm, vias 0 -> 4
- net /Interlock/SW2_4: track 0.00 -> 56.1 mm, vias 0 -> 4
- net /Interlock/SW2_5: track 0.00 -> 54.1 mm, vias 0 -> 4
- net /Interlock/SW2_2: track 0.00 -> 52.6 mm, vias 0 -> 2
- net /Interlock/SW2_6: track 0.00 -> 50.4 mm, vias 0 -> 4
- net /Interlock/SW1_6: track 0.00 -> 44.3 mm, vias 0 -> 2
- net /Interlock/LOAD: track 0.00 -> 43.9 mm, vias 0 -> 4
- net /Interlock/SW1_5: track 0.00 -> 43.8 mm, vias 0 -> 2
- net /Interlock/SW1_4: track 0.00 -> 43.6 mm, vias 0 -> 2
- net /Interlock/SW2_1: track 0.00 -> 40.8 mm, vias 0 -> 3
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- added copper zone on B.Cu, net +1V8
- added copper zone on F.Cu, net +1V8
- added copper zone on B.Cu, net +3V3
- added copper zone on F.Cu, net +3V3

Commit message: final
Parts:
- added C43: 104, lc_lib:0603_C, F.Cu at (70.3, 94.7)
- added J2: Conn_01x01, Connectors:PINTST, F.Cu at (123.5, 109.8)
- added J9: RST, Connectors:PINTST, F.Cu at (63.7, 96.5)
- added R19: 1K, lc_lib:0603_R, F.Cu at (66.6, 94.6)
- added R20: 0, lc_lib:1206_R, F.Cu at (93.0, 64.3)
- added R21: 47K, lc_lib:0603_R, F.Cu at (90.3, 119.4)
- added R22: 47K, lc_lib:0603_R, F.Cu at (94.2, 119.4)
- added R23: 47K, lc_lib:0603_R, F.Cu at (97.9, 119.4)
- added R24: 47K, lc_lib:0603_R, F.Cu at (101.8, 119.3)
- added R38: 47K, lc_lib:0603_R, F.Cu at (105.5, 119.4)
- added R39: 47K, lc_lib:0603_R, F.Cu at (109.4, 119.4)
- added R40: 47K, lc_lib:0603_R, F.Cu at (113.1, 119.3)
- added R41: 47K, lc_lib:0603_R, F.Cu at (117.0, 119.4)
- added R42: 47K, lc_lib:0603_R, F.Cu at (120.8, 119.4)
- added R43: 47K, lc_lib:0603_R, F.Cu at (124.6, 119.4)
- added R60: 47K, lc_lib:0603_R, F.Cu at (128.3, 119.4)
- added R61: 47K, lc_lib:0603_R, F.Cu at (132.1, 119.3)
- added U2: 74HC04, lc_lib:TSSOP-14, F.Cu at (110.7, 115.6)
- added U9: 74HC04, lc_lib:TSSOP-14, F.Cu at (121.6, 115.6)
- moved C10 5.71 mm to (111.5, 74.7)
- moved SC3 1.82 mm to (129.5, 110.6)
- moved J6 0.81 mm to (106.9, 111.7)
- moved R53 0.46 mm to (129.4, 97.8)
- moved F1 0.28 mm to (71.1, 62.7)
- moved D3 0.25 mm to (74.8, 63.8)
- moved U6 0.25 mm to (127.4, 103.1)
- moved C18 0.13 mm to (125.3, 78.1)
- moved R17 0.13 mm to (90.3, 131.3)
- moved C21 0.13 mm to (132.1, 101.5)
Connections:
- C33 pad 1: /Remote/RST -> Net-(C33-Pad1)
- J5 pad 11: /Remote/INT -> Net-(J5-Pad10)
- Q10 pad 1: /Interlock/SEL2_4 -> Net-(Q10-Pad1)
- Q11 pad 1: /Interlock/SEL1_5 -> Net-(Q11-Pad1)
- Q12 pad 1: /Interlock/SEL2_5 -> Net-(Q12-Pad1)
- Q13 pad 1: /Interlock/SEL1_6 -> Net-(Q13-Pad1)
- Q14 pad 1: /Interlock/SEL2_6 -> Net-(Q14-Pad1)
- Q3 pad 1: /Interlock/SEL1_1 -> Net-(Q3-Pad1)
- Q4 pad 1: /Interlock/SEL2_1 -> Net-(Q4-Pad1)
- Q5 pad 1: /Interlock/SEL1_2 -> Net-(Q5-Pad1)
- Q6 pad 1: /Interlock/SEL2_2 -> Net-(Q6-Pad1)
- Q7 pad 1: /Interlock/SEL1_3 -> Net-(Q7-Pad1)
- Q8 pad 1: /Interlock/SEL2_3 -> Net-(Q8-Pad1)
- Q9 pad 1: /Interlock/SEL1_4 -> Net-(Q9-Pad1)
- U1 pad 27: Net-(U1-Pad27) -> /Interlock/CPLDRST
- U4 pad 36: /Remote/RST -> Net-(C33-Pad1)
- U8 pad 3: Net-(C38-Pad1) -> Net-(R20-Pad1)
Routing:
- net /Interlock/SEL1_3: track 35.0 -> 108.8 mm, vias 2 -> 6
- net /Interlock/SEL1_2: track 32.1 -> 79.5 mm, vias 2 -> 9
- net chasis: track 141.4 -> 183.6 mm, vias 86 -> 122
- net Net-(R24-Pad1): track 0.00 -> 35.6 mm, vias 0 -> 4
- net Net-(R21-Pad1): track 0.00 -> 32.8 mm, vias 0 -> 2
- net Net-(R40-Pad1): track 0.00 -> 30.3 mm, vias 0 -> 2
- net +3V3: track 538.4 -> 563.1 mm, vias 46 -> 44
- net Net-(R42-Pad1): track 0.00 -> 23.0 mm, vias 0 -> 2
- net Net-(R39-Pad1): track 0.00 -> 22.1 mm, vias 0 -> 2
- net /Interlock/CPLDRST: track 0.00 -> 21.8 mm, vias 0 -> 2
- net Net-(R22-Pad1): track 0.00 -> 20.2 mm, vias 0 -> 2
- net Net-(R38-Pad1): track 0.00 -> 20.2 mm, vias 0 -> 2
- net /Interlock/SEL2_1: track 32.9 -> 49.9 mm, vias 2 -> 4
- net /Interlock/SEL2_2: track 32.6 -> 49.0 mm, vias 2 -> 4
- net Net-(R23-Pad1): track 0.00 -> 15.3 mm, vias 0 -> 2
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- added copper zone on F.Cu, net Net-(R20-Pad1)
- added copper zone on F.Cu, net chasis
Other:
- net class +3V3: clearance 0.254 -> 0.2032
- net class CH395_GPIO: clearance 0.2032 -> 0.1524
- net class CHASIS: clearance 0.508 -> 0.2032
- net class Default: clearance 0.2032 -> 0.1524
- net class RS485 added: clearance 0.508, trace_width 0.2032, via_dia 0.8, via_drill 0.4
- rule trace_clearance: 0.2032 -> 0.1524
- board text added: "+"
- board text added: "+Freq"
- board text added: "-"
- board text added: "12VDC"
- board text added: "3.3V"
- board text added: "485"
- board text added: "500kHz-2MHz"
- board text added: "6x2 Antenna Switch Control Board V0.2 w/ CPLD Interlock"
- board text added: "A"
- board text added: "B"
- board text added: "CLK"
- board text added: "CPLD RST"
- board text added: "Designed by: Lu, Zening BI4WOP 2019.11.01"
- board text added: "Ethernet"
- board text added: "Feel free to distribute, copy and modify this deisgn"
- board text added: "GND"
- board text added: "IO"
- board text added: "Load"
- board text added: "Power"
- board text added: "RST"
- board text added: "Remote"
- board text added: "SWD"
- board text added: "Zening's Radio Shack BI4WOP"

Commit message: 2024 ver
Routing:
- net /Interlock/SW2_4: track 56.8 -> 53.4 mm
