File: PCB/ControlBoard-2/Interlock.sch (KiCad schematic (older format))
At the start: 76 parts, among them J1 Blaster JTAG, J3 Conn_01x08, J4 Conn_01x08, Q1 8550, Q10 8050, Q11 8050, Q12 8050, Q13 8050, Q14 8050, Q15 8550, Q16 8550, Q17 8550, Q18 8550, Q19 8550, Q2 8550, Q20 8550, Q21 8550, Q22 8550, Q23 8550, Q24 8550, Q25 8550, Q26 8550, Q3 8050, Q4 8050, Q5 8050, Q6 8050, Q7 8050, Q8 8050, Q9 8050, SW1 SRBV170501, SW2 SRBV170501, SW3 LOAD, SW4 REMOTE, U1 EPM240T100

Commit message: Control Board 2 routed
Connections:
- net SW1_1: now also U1.4 (IO1_4); no longer U1.2 (IO1_2)
- net SW1_3: now also U1.2 (IO1_2); no longer U1.4 (IO1_4)
Changed lines of the file:
@@
 	-1   0    0    1
-$EndComp
-$Comp
-L CPLD_Altera:EPM240T100 U1
-U 1 1 5E2DC86A
-P 4100 3500
-F 0 "U1" H 4100 6081 50  0000 C CNN
-F 1 "EPM240T100" H 4100 5990 50  0000 C CNN
-F 2 "lc_lib:LQFP-100_14X14X05P" H 4500 1150 50  0001 L CNN
-F 3 "https://www.altera.com/content/dam/altera-www/global/en_US/pdfs/literature/hb/max2/max2_mii5v1.pdf" H 4100 3500 50  0001 C CNN
-	1    4100 3500
-	1    0    0    -1
 $EndComp
 Wire Wire Line
@@
 $EndComp
 Wire Wire Line
-	1650 1400 3100 1400
-Wire Wire Line
-	1650 1500 3100 1500
-Wire Wire Line
-	1650 1600 3100 1600
-Wire Wire Line
-	1650 1700 3100 1700
-Wire Wire Line
-	1650 1800 3100 1800
-Wire Wire Line
-	1650 1900 3100 1900
-Wire Wire Line
 	1600 2300 3100 2300
 Wire Wire Line
@@
 Text Label 2750 5100 0    50   ~ 0
 SEG1_D
+$Comp
+L CPLD_Altera:EPM240T100 U1
+U 1 1 5E2DC86A
+P 4100 3500
+F 0 "U1" H 4100 6081 50  0000 C CNN
+F 1 "EPM240T100" H 4100 5990 50  0000 C CNN
+F 2 "lc_lib:LQFP-100_14X14X05P" H 4500 1150 50  0001 L CNN
+F 3 "https://www.altera.com/content/dam/altera-www/global/en_US/pdfs/literature/hb/max2/max2_mii5v1.pdf" H 4100 3500 50  0001 C CNN
+	1    4100 3500
+	1    0    0    -1
+$EndComp
+Wire Wire Line
+	3100 1600 2800 1600
+Wire Wire Line
+	3100 1700 2800 1700
+Wire Wire Line
+	3100 1800 2800 1800
+Text Label 2800 1600 0    50   ~ 0
+SW1_1
+Text Label 2800 1500 0    50   ~ 0
+SW1_2
+Text Label 2800 1400 0    50   ~ 0
+SW1_3
+Wire Wire Line
+	2800 1400 3100 1400
+Wire Wire Line
+	2800 1500 3100 1500
+Text Label 2800 1700 0    50   ~ 0
+SW1_4
+Text Label 2800 1800 0    50   ~ 0
+SW1_5
+Text Label 2800 1900 0    50   ~ 0
+SW1_6
+Wire Wire Line
+	2800 1900 3100 1900
 $EndSCHEMATC

Commit message: final
Parts:
- added C43: 104, lc_lib:0603_C, symbol Device:C_Small
- added J9: RST, Connectors:PINTST, symbol Connector_Generic:Conn_01x01
- added R19: 1K, lc_lib:0603_R, symbol Device:R_Small
- added R21, R22, R23, R24, R38, R39, R40, R41, R42, R43, R60, R61: 47K, lc_lib:0603_R, symbol Device:R_Small
- added U2, U9: 74HC04, lc_lib:TSSOP-14, symbol 74xx:74HC04
Connections:
- net +3V3: now also R19.1, U2.14 (VCC), U9.14 (VCC)
- net GND: now also C43.2, U2.7 (GND), U9.7 (GND)
- net SEL1_1: now also U2.1; no longer Q3.1 (B)
- net SEL1_2: now also U2.5; no longer Q5.1 (B)
- net SEL1_3: now also U2.11; no longer Q7.1 (B)
- net SEL1_4: now also U9.1; no longer Q9.1 (B)
- net SEL1_5: now also U9.5; no longer Q11.1 (B)
- net SEL1_6: now also U9.11; no longer Q13.1 (B)
- net SEL2_1: now also U2.3; no longer Q4.1 (B)
- net SEL2_2: now also U2.9; no longer Q6.1 (B)
- net SEL2_3: now also U2.13; no longer Q8.1 (B)
- net SEL2_4: now also U9.3; no longer Q10.1 (B)
- net SEL2_5: now also U9.9; no longer Q12.1 (B)
- net SEL2_6: now also U9.13; no longer Q14.1 (B)
- net CPLDRST: now reaches U1.27 (IO1_27)
- net CPLDRST: now also C43.1, J9.1 (Pin_1), R19.2
- new net: R21.1, U2.2
- new net: R22.1, U2.4
- new net: R23.1, U2.6
- new net: R24.1, U2.8
- new net: R38.1, U2.10
- new net: R39.1, U2.12
- new net: R40.1, U9.2
- new net: R41.1, U9.4
- new net: R42.1, U9.6
- new net: R43.1, U9.8
- new net: R60.1, U9.10
- new net: R61.1, U9.12
- new net: Q3.1 (B), R21.2
- new net: Q4.1 (B), R22.2
- new net: Q5.1 (B), R23.2
- new net: Q6.1 (B), R24.2
- new net: Q7.1 (B), R38.2
- new net: Q8.1 (B), R39.2
- new net: Q9.1 (B), R40.2
- new net: Q10.1 (B), R41.2
- new net: Q11.1 (B), R42.2
- new net: Q12.1 (B), R43.2
- new net: Q13.1 (B), R60.2
- new net: Q14.1 (B), R61.2
Other:
- moved on the sheet: R18
