File: PCB/ControlBoard-2/Power.sch (KiCad schematic (older format))
At the start: 25 parts, among them J8 12VDC, U7 SY8303, U8 AZ1117-3.3

Commit message: final
Parts:
- added R20: 0, lc_lib:1206_R, symbol Device:R_Small
- C40: value 4.7uF 25V -> 2.2uF 50V
Connections:
- net at C38.1, C41.1, L1.2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: now also R20.2; no longer U8.3 (VI)
- new net: R20.1, U8.3 (VI)
Other:
- moved on the sheet: C42
Changed lines of the file:
@@
 L power:+3.3V #PWR058
 U 1 1 5DCA9CAC
-P 6600 1600
-F 0 "#PWR058" H 6600 1450 50  0001 C CNN
-F 1 "+3.3V" H 6615 1773 50  0000 C CNN
-F 2 "" H 6600 1600 50  0001 C CNN
-F 3 "" H 6600 1600 50  0001 C CNN
-	1    6600 1600
+P 7000 1600
+F 0 "#PWR058" H 7000 1450 50  0001 C CNN
+F 1 "+3.3V" H 7015 1773 50  0000 C CNN
+F 2 "" H 7000 1600 50  0001 C CNN
+F 3 "" H 7000 1600 50  0001 C CNN
+	1    7000 1600
 	1    0    0    -1
 $EndComp
@@
 	4800 1750 4800 1700
 Wire Wire Line
-	4800 1700 5250 1700
+	4800 1700 4850 1700
 Wire Wire Line
 	4250 2050 4500 2050
-Wire Wire Line
-	5250 1700 5250 1800
-Connection ~ 5250 1700
 $Comp
 L Device:D_Zener_Small D2
@@
 P 2800 1900
 F 0 "C40" H 2750 1800 50  0000 R CNN
-F 1 "4.7uF 25V" H 2750 1700 50  0000 R CNN
+F 1 "2.2uF 50V" H 2750 1700 50  0000 R CNN
 F 2 "lc_lib:0805_C" H 2800 1900 50  0001 C CNN
 F 3 "~" H 2800 1900 50  0001 C CNN
@@
 Wire Wire Line
 	6050 1700 6250 1700
-Wire Wire Line
-	5250 1700 5450 1700
 $Comp
 L Device:C_Small C42
 U 1 1 5E8455A7
-P 6600 1900
-F 0 "C42" H 6692 1946 50  0000 L CNN
-F 1 "22uF" H 6692 1855 50  0000 L CNN
-F 2 "lc_lib:0805_C" H 6600 1900 50  0001 C CNN
-F 3 "~" H 6600 1900 50  0001 C CNN
-	1    6600 1900
-	1    0    0    -1
-$EndComp
-Wire Wire Line
-	6600 1800 6600 1700
-Wire Wire Line
-	6600 1700 6250 1700
-Connection ~ 6250 1700
+P 7000 1900
+F 0 "C42" H 7092 1946 50  0000 L CNN
+F 1 "22uF" H 7092 1855 50  0000 L CNN
+F 2 "lc_lib:0805_C" H 7000 1900 50  0001 C CNN
+F 3 "~" H 7000 1900 50  0001 C CNN
+	1    7000 1900
+	1    0    0    -1
+$EndComp
+Wire Wire Line
+	7000 1800 7000 1700
 $Comp
 L power:GND #PWR071
 U 1 1 5E84A0BB
-P 6600 2100
-F 0 "#PWR071" H 6600 1850 50  0001 C CNN
-F 1 "GND" H 6605 1927 50  0000 C CNN
-F 2 "" H 6600 2100 50  0001 C CNN
-F 3 "" H 6600 2100 50  0001 C CNN
-	1    6600 2100
-	1    0    0    -1
-$EndComp
-Wire Wire Line
-	6600 2000 6600 2100
+P 7000 2100
+F 0 "#PWR071" H 7000 1850 50  0001 C CNN
+F 1 "GND" H 7005 1927 50  0000 C CNN
+F 2 "" H 7000 2100 50  0001 C CNN
+F 3 "" H 7000 2100 50  0001 C CNN
+	1    7000 2100
+	1    0    0    -1
+$EndComp
+Wire Wire Line
+	7000 2000 7000 2100
 $Comp
 L power:GND #PWR063
@@
 	5750 2000 5750 2100
 Wire Wire Line
-	6600 1600 6600 1700
-Connection ~ 6600 1700
+	7000 1600 7000 1700
+Connection ~ 7000 1700
 Wire Wire Line
 	1900 1700 2200 1700
@@
 Wire Wire Line
 	2200 2100 2200 2150
+$Comp
+L Device:R_Small R20
+U 1 1 5E5140D6
+P 5000 1700
+F 0 "R20" V 4804 1700 50  0000 C CNN
+F 1 "0" V 4895 1700 50  0000 C CNN
+F 2 "lc_lib:1206_R" H 5000 1700 50  0001 C CNN
+F 3 "~" H 5000 1700 50  0001 C CNN
+	1    5000 1700
+	0    1    1    0
+$EndComp
+Connection ~ 6250 1700
+Wire Wire Line
+	6250 1700 7000 1700
+Wire Wire Line
+	5100 1700 5450 1700
+Wire Wire Line
+	4850 1700 4850 1800
+Wire Wire Line
+	4850 1800 5250 1800
+Connection ~ 4850 1700
+Wire Wire Line
+	4850 1700 4900 1700
 $EndSCHEMATC
