File: PCB/RelayBoard-2/AntennaSwitch_6x2_RelayBoard/AntennaSwitch_6x2_RelayBoard.kicad_pcb (KiCad board)
At the start: 2 copper layers, 200 x 90 mm, 42 parts, among them J1 Conn_Coaxial, J10 Conn_01x08, J2 Conn_Coaxial, J3 Conn_Coaxial, J4 Conn_Coaxial, J5 Conn_Coaxial, J6 Conn_Coaxial, J7 Conn_Coaxial, J8 Conn_Coaxial, J9 Conn_01x08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

Commit message: 2024 ver
Routing:
- net /SEL1_6: track 126.8 -> 128.6 mm
- net /SEL1_4: track 87.4 -> 89.0 mm
- net A: track 285.8 -> 287.0 mm
- net GND: vias 304 -> 302
Other:
- board text added: "Shield"
