File: PCB/RelayBoard-3/AntennaSwitch_6x2_RelayBoard/AntennaSwitch_6x2_RelayBoard.sch (KiCad schematic (older format))
At the start: 42 parts, among them J1 Conn_Coaxial, J10 Conn_01x08, J2 Conn_Coaxial, J3 Conn_Coaxial, J4 Conn_Coaxial, J5 Conn_Coaxial, J6 Conn_Coaxial, J7 Conn_Coaxial, J8 Conn_Coaxial, J9 Conn_01x08, K1 G2RL-1-E, K10 G2RL-1-E, K11 G2RL-1-E, K12 G2RL-1-E, K13 G2RL-1-E, K14 G2RL-1-E, K15 G2RL-1-E, K16 G2RL-1-E, K17 G2RL-1-E, K18 G2RL-1-E, K2 G2RL-1-E, K3 G2RL-1-E, K4 G2RL-1-E, K5 G2RL-1-E, K6 G2RL-1-E, K7 G2RL-1-E, K8 G2RL-1-E, K9 G2RL-1-E

Commit message: Start to add support for WebSocket
Connections:
- net A: now also J8.1 (In), K13.4, K13.5, K14.4, K14.5, K15.4, K15.5, K16.4, K16.5, K17.4, K17.5, K18.4, K18.5; no longer J1.1 (In), K1.4, K1.5, K2.4, K2.5, K3.4, K3.5, K4.4, K4.5, K5.4, K5.5, K6.4, K6.5
- net ANT1: now also J7.1 (In), K12.3, K12.6; no longer J2.1 (In), K7.3, K7.6
- net ANT1_A: now also K12.4, K12.5, K6.3, K6.6; no longer K1.3, K1.6, K7.4, K7.5
- net ANT1_B: now also K12.2, K12.7, K18.3, K18.6; no longer K13.3, K13.6, K7.2, K7.7
- net ANT2: now also J6.1 (In), K11.3, K11.6; no longer J3.1 (In), K8.3, K8.6
- net ANT2_A: now also K11.4, K11.5, K5.3, K5.6; no longer K2.3, K2.6, K8.4, K8.5
- net ANT2_B: now also K11.2, K11.7, K17.3, K17.6; no longer K14.3, K14.6, K8.2, K8.7
- net ANT3: now also J5.1 (In), K10.3, K10.6; no longer J4.1 (In), K9.3, K9.6
- net ANT3_A: now also K10.4, K10.5, K4.3, K4.6; no longer K3.3, K3.6, K9.4, K9.5
- net ANT3_B: now also K10.2, K10.7, K16.3, K16.6; no longer K15.3, K15.6, K9.2, K9.7
- net ANT4: now also J4.1 (In), K9.3, K9.6; no longer J5.1 (In), K10.3, K10.6
- net ANT4_A: now also K3.3, K3.6, K9.4, K9.5; no longer K10.4, K10.5, K4.3, K4.6
- net ANT4_B: now also K15.3, K15.6, K9.2, K9.7; no longer K10.2, K10.7, K16.3, K16.6
- net ANT5: now also J3.1 (In), K8.3, K8.6; no longer J6.1 (In), K11.3, K11.6
- net ANT5_A: now also K2.3, K2.6, K8.4, K8.5; no longer K11.4, K11.5, K5.3, K5.6
- net ANT5_B: now also K14.3, K14.6, K8.2, K8.7; no longer K11.2, K11.7, K17.3, K17.6
- net ANT6: now also J2.1 (In), K7.3, K7.6; no longer J7.1 (In), K12.3, K12.6
- net ANT6_A: now also K1.3, K1.6, K7.4, K7.5; no longer K12.4, K12.5, K6.3, K6.6
- net ANT6_B: now also K13.3, K13.6, K7.2, K7.7; no longer K12.2, K12.7, K18.3, K18.6
- net B: now also J1.1 (In), K1.4, K1.5, K2.4, K2.5, K3.4, K3.5, K4.4, K4.5, K5.4, K5.5, K6.4, K6.5; no longer J8.1 (In), K13.4, K13.5, K14.4, K14.5, K15.4, K15.5, K16.4, K16.5, K17.4, K17.5, K18.4, K18.5
- net SEL1_4 renamed SEL2_3
- net SEL1_5 renamed SEL2_2
- net SEL1_6 renamed SEL2_1
Changed lines of the file:
@@
 Connection ~ 9950 700
 Text GLabel 10650 700  2    50   Output ~ 0
-A
+B
 Wire Wire Line
 	2050 2300 2000 2300
@@
 	5000 4100 5000 4400
 Text GLabel 1500 4150 0    50   Output ~ 0
-B
+A
 Wire Wire Line
 	9450 3500 9450 3400
@@
 	1    0    0    -1
 $EndComp
-Text Label 2650 2400 0    50   ~ 0
+Text Label 2650 2400 3    50   ~ 0
+ANT6
+Text Label 4100 2400 3    50   ~ 0
+ANT5
+Text Label 5500 2400 3    50   ~ 0
+ANT4
+Text Label 7000 2400 3    50   ~ 0
+ANT3
+Text Label 8150 2400 3    50   ~ 0
+ANT2
+Text Label 9800 2450 3    50   ~ 0
 ANT1
-Text Label 4150 2400 0    50   ~ 0
-ANT2
-Text Label 5500 2400 0    50   ~ 0
-ANT3
-Text Label 6950 2400 0    50   ~ 0
-ANT4
-Text Label 8150 2400 0    50   ~ 0
-ANT5
-Text Label 9800 2450 0    50   ~ 0
-ANT6
 Text Label 2000 1950 0    50   ~ 0
+ANT6_A
+Text Label 3950 1900 0    50   ~ 0
+ANT5_A
+Text Label 5400 1900 0    50   ~ 0
+ANT4_A
+Text Label 6900 1900 0    50   ~ 0
+ANT3_A
+Text Label 8350 1900 0    50   ~ 0
+ANT2_A
+Text Label 9850 1900 0    50   ~ 0
 ANT1_A
-Text Label 3950 1900 0    50   ~ 0
-ANT2_A
-Text Label 5400 1900 0    50   ~ 0
-ANT3_A
-Text Label 6900 1900 0    50   ~ 0
-ANT4_A
-Text Label 8350 1900 0    50   ~ 0
-ANT5_A
-Text Label 9850 1900 0    50   ~ 0
-ANT6_A
 Text Label 2000 3100 0    50   ~ 0
+ANT6_B
+Text Label 3450 3100 0    50   ~ 0
+ANT5_B
+Text Label 4800 3100 0    50   ~ 0
+ANT4_B
+Text Label 6300 3100 0    50   ~ 0
+ANT3_B
+Text Label 7500 3100 0    50   ~ 0
+ANT2_B
+Text Label 9150 3150 0    50   ~ 0
 ANT1_B
-Text Label 3450 3100 0    50   ~ 0
-ANT2_B
-Text Label 4800 3100 0    50   ~ 0
-ANT3_B
-Text Label 6300 3100 0    50   ~ 0
-ANT4_B
-Text Label 7500 3100 0    50   ~ 0
-ANT5_B
-Text Label 9150 3100 0    50   ~ 0
-ANT6_B
 Connection ~ 7950 4700
 Wire Wire Line
@@
 	4000 6600 4000 6900
 Text Label 5800 6900 1    50   ~ 0
-SEL1_6
+SEL2_1
 Text Label 5600 6900 1    50   ~ 0
-SEL1_5
+SEL2_2
 Text Label 5400 6900 1    50   ~ 0
-SEL1_4
+SEL2_3
 Wire Wire Line
 	3900 6900 3900 6700
